File: Jakarta_R1/Jakarta_R1.kicad_pcb (KiCad board)
At the start: 2 copper layers, 115.2 x 115.2 mm, 84 parts, among them J1 Conn_01x02, J2 USB_C_Receptacle_USB2.0_16P, U1 RP2040, U2 NCP1117-3.3_SOT223, U3 W25Q128JVS, Y1 Crystal_GND24

Commit message: Update Jakarta_R1.kicad_pcb
Routing:
- net Net-(D10-A): track 4.62 -> 57.2 mm
Other:
- board text added: "test"
